Commit message: gripper with two joints working

File: tfm_ws/src/mario_package/robots/quad_arm_default_gripper.urdf (robot description, URDF)
Before this commit: robot fr3, 90 links, 89 joints
Joints:
- joint panda_1_finger_joint2: mimic joint=panda_1_finger_joint1 -> (none)
- joint panda_2_finger_joint2: mimic joint=panda_2_finger_joint1 -> (none)
- joint panda_3_finger_joint2: mimic joint=panda_3_finger_joint1 -> (none)
- joint panda_4_finger_joint2: mimic joint=panda_4_finger_joint1 -> (none)
